File: TxUSB/com_prgm.sch (KiCad schematic (older format))
At the start: 9 parts

Commit message: 
Parts:
- removed D? (x3): DIODE, symbol DIODE
- removed P?: CONN_6, symbol CONN_6
- removed R?: R, symbol R
- added D1, D2, D3: 5V1, symbol ZENER
- added P1: ISP-12PIN, symbol ISP-12PIN
- added Q1: BC547, symbol NPN
- added R1, R6: 4K7, symbol R
- added R2: 10K, symbol R
- R3: renamed from R?; value R -> 10K
- R4, R5: renamed from R?; value R -> 4K7
- gave numbers to parts that had none: 1
Connections:
- net labels added: GND
- wire segments 10 -> 31
- no-connect marks 0 -> 4
Other:
- note removed: "GND"
- note removed: "MISO"
- note removed: "MOSI"
- note removed: "RESET"
- note removed: "SCK"
- note removed: "VCC"
